File: Hardware/KiCad/CaroFocIw/CaroFocIw.kicad_pcb (KiCad board)
At the start: 4 copper layers, 85 x 42 mm, 108 parts, among them J1 Conn_01x04, J10 Conn_01x03, J11 Conn_01x03, J12 Conn_01x03, J13 Conn_01x04, J14 Conn_01x04, J15 Conn_01x04, J16 Conn_01x04, J17 Conn_01x04, J18 Conn_01x04, J19 Conn_01x02, J2 Conn_01x01, J20 Conn_01x02, J3 Conn_01x01, J4 Conn_01x04_MountingPin, J5 Conn_01x02, J6 Conn_01x02, J7 Conn_01x03, J8 Conn_01x03, J9 Conn_01x03, Q1 BSZ013NE2LS5I, Q2 BSZ013NE2LS5I, Q3 BSZ013NE2LS5I, Q4 BSZ013NE2LS5I, Q5 BSZ013NE2LS5I, Q6 BSZ013NE2LS5I, U1 Conn_01x01, U2 TCAN332, U3 STM32F405RGTx, U4 TLE7185-1E, U5 ACS711xEXLT-15AB, U6 AS5048A, U7 ACS711xEXLT-15AB, U8 ACS711xEXLT-15AB, U9 LMR16006YQ3

Commit message: actual version 1.0, several bugfixes and improvements
Parts:
- removed C18: 10μ 6.3V, Capacitor_SMD:C_0603_1608Metric
- removed R14, R15, R16, R6, R7: 10k, Resistor_SMD:R_0603_1608Metric
- removed R2: 100k, Resistor_SMD:R_0603_1608Metric
- removed R4: 1k, Resistor_SMD:R_0603_1608Metric
- C24: footprint Capacitor_SMD:C_0603_1608Metric -> Capacitor_SMD:C_1206_3216Metric
- C9: value 4.7µ 35V -> 10µ 35V; footprint Capacitor_SMD:C_0603_1608Metric -> Capacitor_SMD:C_1206_3216Metric
- D1: value D_Schottky -> D_Schottky 1A
- L1: value 10μ -> 10μ 1A
- L2: value 10μ -> 10μ 100mA
- R10, R11, R13, R5, R8, R9: value 10 -> 4.7
- R17: value 47k -> 56k
- moved R3 2.50 mm to (17.5, 10.5)
- moved C9 2.28 mm to (15.0, 8.60), turned to 0 degrees
- moved C17 1.50 mm to (-1.50, 3.00)
- moved C4 1.50 mm to (-3.50, 3.00), turned to 270 degrees
- moved C10 1.41 mm to (14.0, 6.50), turned to 0 degrees
- moved R17 0.79 mm to (-5.50, 3.00), turned to 90 degrees
- moved C12 0.54 mm to (14.2, 10.5)
- moved R12 0.30 mm to (-1.50, 18.7)
Connections:
- U3 pad 27: (no net) -> /DcLinkVoltageSensing/AnalogOut
- U3 pad 30: /DcLinkVoltageSensing/AnalogOut -> (no net)
- U4 pad 1: (no net) -> GND
- U4 pad 12: Net-(R2-Pad2) -> +3V3
- U4 pad 2: Net-(R6-Pad1) -> /MCU/~GateDriverErr2
- U4 pad 3: Net-(R7-Pad1) -> /MCU/~GateDriverErr1
- U4 pad 34: Net-(R4-Pad2) -> BattA
- U5 pad 4: Net-(R14-Pad2) -> (no net)
- U7 pad 4: Net-(R15-Pad2) -> (no net)
- U8 pad 4: Net-(R16-Pad2) -> (no net)
Routing:
- net /MCU/~GateDriverErr2: track 29.2 -> 52.9 mm
- net /MCU/~GateDriverErr1: track 27.7 -> 51.5 mm
- net Net-(R6-Pad1): track 22.6 -> 0.00 mm
- net Net-(R7-Pad1): track 21.9 -> 0.00 mm
- net Net-(R2-Pad2): track 6.33 -> 0.00 mm
- net /Can/CanL: track 37.0 -> 34.2 mm, vias 0 -> 1
- net Net-(R4-Pad2): track 2.54 -> 0.00 mm
- net Net-(R15-Pad2): track 2.31 -> 0.00 mm
- net Net-(R16-Pad2): track 2.31 -> 0.00 mm
- net Net-(R14-Pad2): track 2.31 -> 0.00 mm
- net Net-(C10-Pad1): track 4.62 -> 2.61 mm
- net BattA: track 67.0 -> 65.4 mm
- net +3V3: track 26.2 -> 27.6 mm, vias 9 -> 10
- net 3.3VA_W: track 5.11 -> 4.25 mm, vias 1 -> 0
- net 3.3VA_V: track 5.11 -> 4.25 mm, vias 1 -> 0
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- added copper zone on F.Cu, net 3.3VA_U
- added copper zone on F.Cu, net 3.3VA_V
- added copper zone on In1.Cu, net GNDPWR
- removed copper zone on In2.Cu, net 3.3VA_U
- removed copper zone on In2.Cu, net 3.3VA_V
- removed copper zone on In2.Cu, net 3.3VA_W

Commit message: Actual actual version 1.0, some minor changes. PCBs ordered.
Parts:
- J10, J12, J8: footprint Connector_PinHeader_2.00mm:PinHeader_1x03_P2.00mm_Vertical -> Connector_PinSocket_2.00mm:PinSocket_1x03_P2.00mm_Vertical
- J14, J16, J18: footprint Connector_PinHeader_2.00mm:PinHeader_1x04_P2.00mm_Vertical -> Connector_PinSocket_2.00mm:PinSocket_1x04_P2.00mm_Vertical
- J20, J6: footprint Connector_PinHeader_2.00mm:PinHeader_1x02_P2.00mm_Vertical -> Connector_PinSocket_2.00mm:PinSocket_1x02_P2.00mm_Vertical
Connections:
- U3 pad 40: (no net) -> /Encoder/~EncoderCs
Routing:
- net /Encoder/~EncoderCs: track 13.5 -> 15.0 mm
